Commit message: backup

File: urdf/inc/ur10_macro.xacro (robot description, xacro)
@@ -19,8 +19,8 @@
   <xacro:macro name="ur10_robot" params="
    prefix
-   joint_limits_parameters_file:='$(find nrs_vision_rviz)/config/joint_limits.yaml'
-   kinematics_parameters_file:='$(find nrs_vision_rviz)/config/default_kinematics.yaml'
-   physical_parameters_file:='$(find nrs_vision_rviz)/config/physical_parameters.yaml'
-   visual_parameters_file:='$(find nrs_vision_rviz)/config/visual_parameters.yaml'
+   joint_limits_parameters_file:='$(find nrs_path_planning)/config/joint_limits.yaml'
+   kinematics_parameters_file:='$(find nrs_path_planning)/config/default_kinematics.yaml'
+   physical_parameters_file:='$(find nrs_path_planning)/config/physical_parameters.yaml'
+   visual_parameters_file:='$(find nrs_path_planning)/config/visual_parameters.yaml'
    transmission_hw_interface:=hardware_interface/PositionJointInterface
    safety_limits:=false
@@ -28,5 +28,5 @@
    safety_k_position:=20"
   >
-    <xacro:include filename="$(find nrs_vision_rviz)/urdf/inc/ur_macro.xacro"/>
+    <xacro:include filename="$(find nrs_path_planning)/urdf/inc/ur_macro.xacro"/>
     <xacro:ur_robot
       prefix="${prefix}"

File: urdf/inc/ur_common.xacro (robot description, xacro)
@@ -21,5 +21,5 @@
           However, users MUST NOT rely on these properties, their contents or
           their names.
-          This macro is NOT part of the public API of the nrs_vision_rviz pkg,
+          This macro is NOT part of the public API of the nrs_path_planning pkg,
           and as such should be considered to be for internal use only.
   -->

File: urdf/inc/ur_macro.xacro (robot description, xacro)
@@ -42,6 +42,6 @@
      - Muhammad Asif Rana
   -->
-  <xacro:include filename="$(find nrs_vision_rviz)/urdf/inc/ur_transmissions.xacro" />
-  <xacro:include filename="$(find nrs_vision_rviz)/urdf/inc/ur_common.xacro" />
+  <xacro:include filename="$(find nrs_path_planning)/urdf/inc/ur_transmissions.xacro" />
+  <xacro:include filename="$(find nrs_path_planning)/urdf/inc/ur_common.xacro" />
   <xacro:macro name="ur_robot" params="
     prefix

File: urdf/testbed.xacro (robot description, xacro)
@@ -2,5 +2,5 @@
 <robot name="ur10_robot" xmlns:xacro="http://www.ros.org/wiki/xacro">
   <!-- Include the UR10 robot description -->
-  <xacro:include filename="$(find nrs_vision_rviz)/urdf/ur10.xacro" />
+  <xacro:include filename="$(find nrs_path_planning)/urdf/ur10.xacro" />
   <!-- Define the testbed link -->
   <link name="testbed">
@@ -32,5 +32,5 @@
     <visual>
       <geometry>
-        <mesh filename="package://nrs_vision_rviz/mesh/ur10_tooltip.stl" />
+        <mesh filename="package://nrs_path_planning/mesh/ur10_tooltip.stl" />
       </geometry>
       <material name="tooltip_gray">
@@ -40,5 +40,5 @@
     <collision>
       <geometry>
-        <mesh filename="package://nrs_vision_rviz/mesh/ur10_tooltip.stl" />
+        <mesh filename="package://nrs_path_planning/mesh/ur10_tooltip.stl" />
       </geometry>
       <material name="tooltip_gray">
@@ -50,5 +50,5 @@
     <visual>
       <geometry>
-        <mesh filename="package://nrs_vision_rviz/mesh/lid_wrap.stl" />
+        <mesh filename="package://nrs_path_planning/mesh/lid_wrap.stl" />
       </geometry>
       <material name="light_blue">
@@ -58,5 +58,5 @@
     <collision>
       <geometry>
-        <mesh filename="package://nrs_vision_rviz/mesh/lid_wrap.stl" />
+        <mesh filename="package://nrs_path_planning/mesh/lid_wrap.stl" />
       </geometry>
       <material name="light_blue">

File: urdf/ur.xacro (robot description, xacro)
@@ -2,5 +2,5 @@
 <robot xmlns:xacro="http://wiki.ros.org/xacro" name="$(arg robot_model)_robot">
    <!-- import main macro -->
-   <xacro:include filename="$(find nrs_vision_rviz)/urdf/inc/ur_macro.xacro"/>
+   <xacro:include filename="$(find nrs_path_planning)/urdf/inc/ur_macro.xacro"/>
    <!-- parameters -->
    <xacro:arg name="joint_limit_params" default=""/>

File: urdf/ur10.xacro (robot description, xacro)
@@ -14,5 +14,5 @@
     Refer to 'inc/ur_macro.xacro' for more information.
   -->
-  <xacro:include filename="$(find nrs_vision_rviz)/urdf/inc/ur10_macro.xacro"/>
+  <xacro:include filename="$(find nrs_path_planning)/urdf/inc/ur10_macro.xacro"/>
   <xacro:ur10_robot prefix="" />
 </robot>

Commit message: backup

File: urdf/inc/ur10_macro.xacro (robot description, xacro)
@@ -19,8 +19,8 @@
   <xacro:macro name="ur10_robot" params="
    prefix
-   joint_limits_parameters_file:='$(find nrs_path_planning)/config/joint_limits.yaml'
-   kinematics_parameters_file:='$(find nrs_path_planning)/config/default_kinematics.yaml'
-   physical_parameters_file:='$(find nrs_path_planning)/config/physical_parameters.yaml'
-   visual_parameters_file:='$(find nrs_path_planning)/config/visual_parameters.yaml'
+   joint_limits_parameters_file:='$(find nrs_vision_rviz)/config/joint_limits.yaml'
+   kinematics_parameters_file:='$(find nrs_vision_rviz)/config/default_kinematics.yaml'
+   physical_parameters_file:='$(find nrs_vision_rviz)/config/physical_parameters.yaml'
+   visual_parameters_file:='$(find nrs_vision_rviz)/config/visual_parameters.yaml'
    transmission_hw_interface:=hardware_interface/PositionJointInterface
    safety_limits:=false
@@ -28,5 +28,5 @@
    safety_k_position:=20"
   >
-    <xacro:include filename="$(find nrs_path_planning)/urdf/inc/ur_macro.xacro"/>
+    <xacro:include filename="$(find nrs_vision_rviz)/urdf/inc/ur_macro.xacro"/>
     <xacro:ur_robot
       prefix="${prefix}"

File: urdf/inc/ur_common.xacro (robot description, xacro)
@@ -21,5 +21,5 @@
           However, users MUST NOT rely on these properties, their contents or
           their names.
-          This macro is NOT part of the public API of the nrs_path_planning pkg,
+          This macro is NOT part of the public API of the nrs_vision_rviz pkg,
           and as such should be considered to be for internal use only.
   -->

File: urdf/inc/ur_macro.xacro (robot description, xacro)
@@ -42,6 +42,6 @@
      - Muhammad Asif Rana
   -->
-  <xacro:include filename="$(find nrs_path_planning)/urdf/inc/ur_transmissions.xacro" />
-  <xacro:include filename="$(find nrs_path_planning)/urdf/inc/ur_common.xacro" />
+  <xacro:include filename="$(find nrs_vision_rviz)/urdf/inc/ur_transmissions.xacro" />
+  <xacro:include filename="$(find nrs_vision_rviz)/urdf/inc/ur_common.xacro" />
   <xacro:macro name="ur_robot" params="
     prefix

File: urdf/testbed.xacro (robot description, xacro)
@@ -2,5 +2,5 @@
 <robot name="ur10_robot" xmlns:xacro="http://www.ros.org/wiki/xacro">
   <!-- Include the UR10 robot description -->
-  <xacro:include filename="$(find nrs_path_planning)/urdf/ur10.xacro" />
+  <xacro:include filename="$(find nrs_vision_rviz)/urdf/ur10.xacro" />
   <!-- Define the testbed link -->
   <link name="testbed">
@@ -32,9 +32,5 @@
     <visual>
       <geometry>
-<<<<<<< HEAD
         <mesh filename="package://nrs_vision_rviz/mesh/UR_EE_tool.stl" />
-=======
-        <mesh filename="package://nrs_path_planning/mesh/ur10_tooltip.stl" />
->>>>>>> 745743660d549b29ec120686157a19684c5f67e3
       </geometry>
       <material name="tooltip_gray">
@@ -44,9 +40,5 @@
     <!-- <collision>
       <geometry>
-<<<<<<< HEAD
         <mesh filename="package://nrs_vision_rviz/mesh/UR_EE_tool.stl" />
-=======
-        <mesh filename="package://nrs_path_planning/mesh/ur10_tooltip.stl" />
->>>>>>> 745743660d549b29ec120686157a19684c5f67e3
       </geometry>
       <material name="tooltip_gray">
@@ -58,5 +50,5 @@
     <visual>
       <geometry>
-        <mesh filename="package://nrs_path_planning/mesh/lid_wrap.stl" />
+        <mesh filename="package://nrs_vision_rviz/mesh/lid_wrap.stl" />
       </geometry>
       <material name="light_blue">
@@ -66,5 +58,5 @@
     <collision>
       <geometry>
-        <mesh filename="package://nrs_path_planning/mesh/lid_wrap.stl" />
+        <mesh filename="package://nrs_vision_rviz/mesh/lid_wrap.stl" />
       </geometry>
       <material name="light_blue">

File: urdf/ur.xacro (robot description, xacro)
@@ -2,5 +2,5 @@
 <robot xmlns:xacro="http://wiki.ros.org/xacro" name="$(arg robot_model)_robot">
    <!-- import main macro -->
-   <xacro:include filename="$(find nrs_path_planning)/urdf/inc/ur_macro.xacro"/>
+   <xacro:include filename="$(find nrs_vision_rviz)/urdf/inc/ur_macro.xacro"/>
    <!-- parameters -->
    <xacro:arg name="joint_limit_params" default=""/>

File: urdf/ur10.xacro (robot description, xacro)
@@ -14,5 +14,5 @@
     Refer to 'inc/ur_macro.xacro' for more information.
   -->
-  <xacro:include filename="$(find nrs_path_planning)/urdf/inc/ur10_macro.xacro"/>
+  <xacro:include filename="$(find nrs_vision_rviz)/urdf/inc/ur10_macro.xacro"/>
   <xacro:ur10_robot prefix="" />
 </robot>
