Commit message: backup

File: urdf/inc/ur_common.xacro (robot description, xacro)
@@ -21,5 +21,5 @@
           However, users MUST NOT rely on these properties, their contents or
           their names.
-          This macro is NOT part of the public API of the nrs_vision_rviz pkg,
+          This macro is NOT part of the public API of the ur_description pkg,
           and as such should be considered to be for internal use only.
   -->

File: urdf/testbed.xacro (robot description, xacro)
@@ -1,6 +1,6 @@
 <?xml version="1.0"?>
-<robot name="ur10_robot" xmlns:xacro="http://www.ros.org/wiki/xacro">
+<robot name="ur10e_robot" xmlns:xacro="http://www.ros.org/wiki/xacro">
   <!-- Include the UR10 robot description -->
-  <xacro:include filename="$(find nrs_vision_rviz)/urdf/ur10.xacro" />
+  <xacro:include filename="$(find nrs_vision_rviz)/urdf/ur10e.xacro" />
   <!-- Define the testbed link -->
   <link name="testbed">
@@ -29,8 +29,8 @@
     </inertial>
   </link>
-  <link name="UR_EE_tool">
+  <link name="UR10e_roboworld_tooltip_m">
     <visual>
       <geometry>
-        <mesh filename="package://nrs_vision_rviz/mesh/UR_EE_tool.stl" />
+        <mesh filename="package://nrs_vision_rviz/mesh/UR10e_roboworld_tooltip_m.stl" />
       </geometry>
       <material name="tooltip_gray">
@@ -40,5 +40,5 @@
     <collision>
       <geometry>
-        <mesh filename="package://nrs_vision_rviz/mesh/UR_EE_tool.stl" />
+        <mesh filename="package://nrs_vision_rviz/mesh/UR10e_roboworld_tooltip_m.stl" />
       </geometry>
       <material name="tooltip_gray">
@@ -74,5 +74,5 @@
   <joint name="tooltip_joint" type="fixed">
     <parent link="wrist_3_link" />
-    <child link="UR_EE_tool" />
+    <child link="UR10e_roboworld_tooltip_m" />
     <origin xyz="0 0 0.0" rpy="0 0 0" />
   </joint>
