Commit message: update

File: urdf/inc/ur_macro.xacro (robot description, xacro)
@@ -215,5 +215,5 @@
            link/frame) to introduce the necessary rotation over Z (of pi rad).
       -->
-      <origin xyz="0 0 0" rpy="0 0 0" />
+      <origin xyz="0 0 0" rpy="0 0 ${pi}" />
     </joint>
     <joint name="${prefix}shoulder_pan_joint" type="revolute">

Commit message: update

File: urdf/inc/ur_macro.xacro (robot description, xacro)
@@ -10,5 +10,5 @@
     This file models the base kinematic chain of a UR robot, which then gets
     parameterised by various configuration files to convert it into a UR3(e),
-    UR5(e), UR10(e) or UR16e.
+    UR5(e), UR10(e), UR16e, UR20 or UR30.
     NOTE: the default kinematic parameters (ie: link lengths, frame locations,
     offets, etc) do not correspond to any particular robot. They are defaults
@@ -42,6 +42,6 @@
      - Muhammad Asif Rana
   -->
-  <xacro:include filename="$(find nrs_path)/urdf/inc/ur_transmissions.xacro" />
-  <xacro:include filename="$(find nrs_path)/urdf/inc/ur_common.xacro" />
+  <xacro:include filename="$(find nrs_robot)/urdf/inc/ur_transmissions.xacro" />
+  <xacro:include filename="$(find nrs_robot)/urdf/inc/ur_common.xacro" />
   <xacro:macro name="ur_robot" params="
     prefix
@@ -215,5 +215,5 @@
            link/frame) to introduce the necessary rotation over Z (of pi rad).
       -->
-      <origin xyz="0 0 0" rpy="0 0 ${pi}" />
+      <origin xyz="0 0 0" rpy="0 0 0" />
     </joint>
     <joint name="${prefix}shoulder_pan_joint" type="revolute">

File: urdf/testbed.xacro (robot description, xacro)
@@ -1,6 +1,6 @@
 <?xml version="1.0"?>
-<robot name="ur10e_robot" xmlns:xacro="http://www.ros.org/wiki/xacro">
+<robot name="ur10_robot" xmlns:xacro="http://www.ros.org/wiki/xacro">
   <!-- Include the UR10 robot description -->
-  <xacro:include filename="$(find nrs_path)/urdf/ur10e.xacro" />
+  <xacro:include filename="$(find nrs_path)/urdf/ur10.xacro" />
   <!-- Define the testbed link -->
   <link name="testbed">
