Commit message: backup ompl & tooltip

File: urdf/testbed.xacro (robot description, xacro)
@@ -50,8 +50,8 @@
     <visual>
       <geometry>
-        <mesh filename="package://nrs_vision_rviz/mesh/fenda_wrap.stl"/>
+        <mesh filename="package://nrs_vision_rviz/mesh/lid_wrap.stl"/>
       </geometry>
-      <material name="gray">
-        <color rgba="0.5 0.5 0.5 1.0" />
+      <material name="light_blue">
+        <color rgba="0.57 0.81 0.92 1.0" />
       </material>
     </visual>

Commit message: ompl l blending&projection

File: urdf/testbed.xacro (robot description, xacro)
@@ -10,6 +10,6 @@
         <box size="0.84 1.24 0.9"/> <!-- 840mm x 1240mm x 900mm -->
       </geometry>
-      <material name="gray">
-        <color rgba="0.5 0.5 0.5 1.0" />
+      <material name="testbed_gray">
+        <color rgba="0.5 0.5 0.5 0.5" />
       </material>
     </visual>
@@ -17,8 +17,8 @@
       <origin xyz="0.3 0.5 -0.45" rpy="0 0 0" />
       <geometry>
-        <box size="0.84 1.24 0.9"/> <!-- 840mm x 1240mm x 900mm -->
+        <box size="0.84 1.24 0.9"/>
       </geometry>
-      <material name="gray">
-        <color rgba="0.5 0.5 0.5 1.0" />
+      <material name="testbed_gray">
+        <color rgba="0.5 0.5 0.5 0.5" />
       </material>
     </collision>
@@ -34,5 +34,5 @@
         <mesh filename="package://nrs_vision_rviz/mesh/ur10_tooltip.stl"/>
       </geometry>
-      <material name="gray">
+      <material name="tooltip_gray">
         <color rgba="0.5 0.5 0.5 1.0" />
       </material>
@@ -42,5 +42,5 @@
         <mesh filename="package://nrs_vision_rviz/mesh/ur10_tooltip.stl"/>
       </geometry>
-      <material name="gray">
+      <material name="tooltip_gray">
         <color rgba="0.5 0.5 0.5 1.0" />
       </material>
@@ -71,5 +71,5 @@
     <origin xyz="0 0 0" rpy="0 0 -0.7853981633974483" /> <!-- 45 degrees in radians -->
   </joint>
-  <!-- Define a fixed joint to attach the testbed to the base link -->
+  <!-- Define a fixed joint to attach the tooltip to the wrist_3_link -->
   <joint name="tooltip_joint" type="fixed">
     <parent link="wrist_3_link" />

Commit message: backup

File: urdf/testbed.xacro (robot description, xacro)
@@ -56,5 +56,5 @@
       </material>
     </visual>
-    <!-- <collision>
+     <collision>
       <geometry>
         <mesh filename="package://nrs_vision_rviz/mesh/sample_wrap.stl"/>
@@ -63,5 +63,5 @@
         <color rgba="0.5 0.5 0.5 1.0" />
       </material>
-    </collision> -->
+    </collision>
   </link>
   <!-- Define a fixed joint to attach the testbed to the base link -->

Commit message: projection mode: z-projection

File: urdf/testbed.xacro (robot description, xacro)
@@ -53,13 +53,13 @@
       </geometry>
       <material name="light_blue">
-        <color rgba="0.57 0.81 0.92 1.0" />
+        <color rgba="0.57 0.81 0.92 0.5" />
       </material>
     </visual>
      <collision>
       <geometry>
-        <mesh filename="package://nrs_vision_rviz/mesh/sample_wrap.stl"/>
+        <mesh filename="package://nrs_vision_rviz/mesh/lid_wrap.stl"/>
       </geometry>
-      <material name="gray">
-        <color rgba="0.5 0.5 0.5 1.0" />
+      <material name="light_blue">
+        <color rgba="0.57 0.81 0.92 0.5" />
       </material>
     </collision>

Commit message: geodesic + hermite combine

File: urdf/testbed.xacro (robot description, xacro)
@@ -8,5 +8,5 @@
       <origin xyz="0.3 0.5 -0.45" rpy="0 0 0" />
       <geometry>
-        <box size="0.84 1.24 0.9"/> <!-- 840mm x 1240mm x 900mm -->
+        <box size="0.84 1.24 0.9" /> <!-- 840mm x 1240mm x 900mm -->
       </geometry>
       <material name="testbed_gray">
@@ -17,5 +17,5 @@
       <origin xyz="0.3 0.5 -0.45" rpy="0 0 0" />
       <geometry>
-        <box size="0.84 1.24 0.9"/>
+        <box size="0.84 1.24 0.9" />
       </geometry>
       <material name="testbed_gray">
@@ -32,5 +32,5 @@
     <visual>
       <geometry>
-        <mesh filename="package://nrs_vision_rviz/mesh/ur10_tooltip.stl"/>
+        <mesh filename="package://nrs_vision_rviz/mesh/ur10_tooltip.stl" />
       </geometry>
       <material name="tooltip_gray">
@@ -40,5 +40,5 @@
     <collision>
       <geometry>
-        <mesh filename="package://nrs_vision_rviz/mesh/ur10_tooltip.stl"/>
+        <mesh filename="package://nrs_vision_rviz/mesh/ur10_tooltip.stl" />
       </geometry>
       <material name="tooltip_gray">
@@ -50,5 +50,5 @@
     <visual>
       <geometry>
-        <mesh filename="package://nrs_vision_rviz/mesh/lid_wrap.stl"/>
+        <mesh filename="package://nrs_vision_rviz/mesh/lid_wrap.stl" />
       </geometry>
       <material name="light_blue">
@@ -56,7 +56,7 @@
       </material>
     </visual>
-     <collision>
+    <collision>
       <geometry>
-        <mesh filename="package://nrs_vision_rviz/mesh/lid_wrap.stl"/>
+        <mesh filename="package://nrs_vision_rviz/mesh/lid_wrap.stl" />
       </geometry>
       <material name="light_blue">

Commit message: backup

File: urdf/testbed.xacro (robot description, xacro)
@@ -29,8 +29,8 @@
     </inertial>
   </link>
-  <link name="tooltip">
+  <link name="UR_EE_tool">
     <visual>
       <geometry>
-        <mesh filename="package://nrs_vision_rviz/mesh/ur10_tooltip.stl" />
+        <mesh filename="package://nrs_vision_rviz/mesh/UR_EE_tool.stl" />
       </geometry>
       <material name="tooltip_gray">
@@ -38,12 +38,12 @@
       </material>
     </visual>
-    <collision>
+    <!-- <collision>
       <geometry>
-        <mesh filename="package://nrs_vision_rviz/mesh/ur10_tooltip.stl" />
+        <mesh filename="package://nrs_vision_rviz/mesh/UR_EE_tool.stl" />
       </geometry>
       <material name="tooltip_gray">
         <color rgba="0.5 0.5 0.5 1.0" />
       </material>
-    </collision>
+    </collision> -->
   </link>
   <link name="workpiece">
@@ -74,6 +74,6 @@
   <joint name="tooltip_joint" type="fixed">
     <parent link="wrist_3_link" />
-    <child link="tooltip" />
-    <origin xyz="0 0 0" rpy="0 0 -1.5707963267948966" />
+    <child link="UR_EE_tool" />
+    <origin xyz="0 0 0.0" rpy="0 0 0" />
   </joint>
   <!-- Define a fixed joint to attach the workpiece to the base link -->

Commit message: fix geodesicsubtract function

File: urdf/testbed.xacro (robot description, xacro)
@@ -38,5 +38,5 @@
       </material>
     </visual>
-    <!-- <collision>
+    <collision>
       <geometry>
         <mesh filename="package://nrs_vision_rviz/mesh/UR_EE_tool.stl" />
@@ -45,10 +45,10 @@
         <color rgba="0.5 0.5 0.5 1.0" />
       </material>
-    </collision> -->
+    </collision>
   </link>
   <link name="workpiece">
     <visual>
       <geometry>
-        <mesh filename="package://nrs_vision_rviz/mesh/lid_wrap.stl" />
+        <mesh filename="package://nrs_vision_rviz/mesh/fenda_wrap.stl" />
       </geometry>
       <material name="light_blue">
@@ -56,12 +56,12 @@
       </material>
     </visual>
-    <collision>
+    <!-- <collision>
       <geometry>
-        <mesh filename="package://nrs_vision_rviz/mesh/lid_wrap.stl" />
+        <mesh filename="package://nrs_vision_rviz/mesh/fenda_wrap.stl" />
       </geometry>
       <material name="light_blue">
         <color rgba="0.57 0.81 0.92 0.5" />
       </material>
-    </collision>
+    </collision> -->
   </link>
   <!-- Define a fixed joint to attach the testbed to the base link -->

Commit message: backup

File: urdf/testbed.xacro (robot description, xacro)
@@ -50,5 +50,5 @@
     <visual>
       <geometry>
-        <mesh filename="package://nrs_vision_rviz/mesh/fenda_wrap.stl" />
+        <mesh filename="package://nrs_vision_rviz/mesh/lid_wrap.stl" />
       </geometry>
       <material name="light_blue">
@@ -58,5 +58,5 @@
     <!-- <collision>
       <geometry>
-        <mesh filename="package://nrs_vision_rviz/mesh/fenda_wrap.stl" />
+        <mesh filename="package://nrs_vision_rviz/mesh/lid_wrap.stl" />
       </geometry>
       <material name="light_blue">

Commit message: add readme

File: urdf/testbed.xacro (robot description, xacro)
@@ -50,5 +50,5 @@
     <visual>
       <geometry>
-        <mesh filename="package://nrs_vision_rviz/mesh/lid_wrap.stl" />
+        <mesh filename="package://nrs_vision_rviz/mesh/fenda_wrap.stl" />
       </geometry>
       <material name="light_blue">
@@ -58,5 +58,5 @@
     <!-- <collision>
       <geometry>
-        <mesh filename="package://nrs_vision_rviz/mesh/lid_wrap.stl" />
+        <mesh filename="package://nrs_vision_rviz/mesh/fenda_wrap.stl" />
       </geometry>
       <material name="light_blue">
