Commit message: bug fix

File: urdf/cad_model.xacro (robot description, xacro)
@@ -7,5 +7,5 @@
     <inertial>
       <mass value="0.1"/>
-      <origin xyz="0 0 0" rpy="0 0 0"/>
+      <origin xyz="0 0 0" rpy="0 0 ${pi}"/>
       <inertia ixx="0.1" ixy="0.0" ixz="0.0" iyy="0.1" iyz="0.0" izz="0.1"/>
     </inertial>

File: urdf/scan_model.xacro (robot description, xacro)
@@ -35,5 +35,5 @@
       <parent link="cad_model"/>
       <child link="scan_model"/>
-    <origin xyz="0.7612783054351273 -0.03097931096065283 0.12363673620305149" rpy="0.024916701375427223 0.013877853294511456 2.3236770153618296" />
+    <origin xyz="0.6632968380343811 0.14823617988307086 0.02038985171070404" rpy="0.01109268636821642 0.0012672906445020703 -1.598243791705674" />
     </joint>
   </xacro:macro>
